Commit message: urdff

File: src/bumperbot_description/urdf/bumperbot.urdf (robot description, URDF)
Before this commit: robot bumperbot, 5 links, 5 joints
Links:
- added link caster_front_link; visual mesh filename=package://bumperbot_description/meshes/caster_front_link.STL
Joints:
- removed joint base_name
- added joint base_joint: type fixed, parent base_footprint, child base_link, origin xyz=0.0 0.0 0.033 rpy=0.0 0.0 0.0
- joint wheel_right_joint: parent base_footprint -> base_link
